Commit message: Modify to work with gazebo 11.

File: urdf/gimbal.urdf.xacro (robot description, xacro)
@@ -1,11 +1,12 @@
 <?xml version="1.0"?>
-<robot xmlns:xacro="http://www.ros.org/wiki/xacro">
-    <xacro:include filename="$(find dji_m100_description)/urdf/gimbal_joints.xacro"/>
+<robot xmlns:xacro="http://www.ros.org/wiki/xacro" name="dji_m100_gimbal">
+    <xacro:include filename="$(find dji_m100_description)/urdf/gimbal_joints.xacro" />
     <xacro:property name="M_PI" value="3.14"/>
     <material name="black">
         <color rgba="0 0 0 1"/>
     </material>
-    <xacro:macro name="dji_m100_gimbal">
+    <xacro:macro name="dji_m100_gimbal" params="*origin">
         <joint name="gimbal_base_joint" type="fixed">
+            <xacro:insert_block name="origin" />
             <parent link="base_link"/>
             <child link="gimbal_base_plate" />
@@ -33,5 +34,5 @@
             </inertial>
         </link>
-         <revolute_gimbal_joint
+         <xacro:revolute_gimbal_joint
             name="gimbal_roll_joint"
             parent="gimbal_base_plate"
@@ -54,5 +55,5 @@
             </visual>
         </link>
-        <revolute_gimbal_joint
+        <xacro:revolute_gimbal_joint
             name="gimbal_pitch_joint"
             parent="gimbal_roll_link"
@@ -75,5 +76,5 @@
             </visual>
         </link>
-        <revolute_gimbal_joint
+        <xacro:revolute_gimbal_joint
             name="gimbal_yaw_joint"
             parent="gimbal_pitch_link"
@@ -97,8 +98,8 @@
             </visual>
         </link>
-        <gazebo>
+        <!-- <gazebo>
             <plugin name="gazebo_ros_control" filename="libgazebo_ros_control.so">
             </plugin>
-        </gazebo>
+        </gazebo> -->
         <gazebo reference="gimbal_base_plate">
             <material>Gazebo/FlatBlack</material>
